File: PROYEK_BMS_NUVOTON.kicad_sch (KiCad schematic)
At the start: 257 parts, among them J1 Conn_01x23_Pin, J2 Conn_01x04_Pin, J3 USB_B_Micro, J4 Screw_Terminal_01x02, Q1 NPN, Q17 Q_NMOS_GSD, Q18 Q_NMOS_GSD, Q19 Q_NMOS_GSD, Q20 Q_NMOS_GSD, Q21 Q_NMOS_GSD, Q22 Q_NMOS_GSD, Q23 Q_NMOS_GSD, Q24 Q_NMOS_GSD, Q25 Q_NMOS_GSD, Q26 Q_NMOS_GSD, Q27 Q_NMOS_GSD, Q28 Q_NMOS_GSD, Q29 Q_NMOS_GSD, Q30 Q_NMOS_GSD, Q31 Q_NMOS_GSD, Q32 Q_NMOS_GSD, Q33 Q_NMOS_GSD, Q34 Q_NMOS_GSD, Q35 Q_NMOS_GSD, Q36 Q_NMOS_GSD, Q37 Q_NMOS_GSD, Q38 Q_NMOS_GSD, Q5 NMOS, Q6 NMOS, SW1 SW_SPDT, SW2 SW_Push, SW3 SW_SPDT, U1 KA49522, U2 TL431DBZ, U4 STM32F072RBTx, U5 SN65HVD230, U6 AP7370-33SA-7, Y1 8M,SMD, Y2 32.768k,SMD

Commit message: revision 2, 12 error fix on bms connection with STM32, USB circuit need some adjustment
Parts:
- added C23 (x2): 0.1u, Capacitor_SMD:C_0805_2012Metric, symbol Device:C
- added C49: 0.1 uF, symbol Device:C
- added CVBAT1: 1uF, symbol Device:C
- added DVBAT1: NHP120SFT3G, symbol Device:D
- added R135, R136: NTC10k, Resistor_SMD:R_0603_1608Metric, symbol Device:R
- added R137: 75M, Resistor_SMD:R_0805_2012Metric, symbol Device:R
- added RVBAT1, RVBAT2: 100, symbol Device:R
- added SW4: SW_Push, symbol Switch:SW_Push
- C1: value 2.2u -> 4.7u
- C12, C3: value 100n -> 1n
- R1: value NTC10k -> 47k
- R18: value R -> 47k
- R2: value 100 -> 30k
Connections:
- net C0: now also C11.1; no longer C11.2
- net CN4_C22: now also CVBAT1.2, DVBAT1.2 (A), RVBAT1.1, RVBAT2.2
- net CN4_C7: now also R149.1
- net GND: now also C11.2, R11.2, R13.2, R7.2, R9.2, C23.2, C23.2, C49.2, R135.2, R136.2; no longer C11.1, R11.1, R13.1, R7.1, R9.1, U1.12 (REGSEL)
- net GNDA: now also CVBAT1.1
- net SRN: now also C23.1
- net SRP: now also C23.1
- net TMON1: now also C3.1, R1.1, U1.3 (TMONI1), R135.1; no longer C12.1, R18.1
- net TMON2: now also C12.1, R18.1, R136.1; no longer C3.1, R1.1, U1.3 (TMONI1)
- net VDD55: now also U1.12 (REGSEL)
- net VPACK+: now also SW4.2
- net VPACK-: now also R11.1, R13.1, R7.1, R9.1; no longer R11.2, R13.2, R7.2, R9.2
- net at U1.18 (VPC): now also R137.2
- net BMS_5V renamed BMS_3.3V
- net BMS_3.3V: now also C49.1
- new net: DVBAT1.1 (K), RVBAT1.2, RVBAT2.1
- new net: R137.1, SW4.1
- no-connect marks 9 -> 8
Other:
- note added: "2. Suggest place VDD18 output Cap near BMIC for best ESD/EMC consideration"
- note added: "2. Wide line width to be drawn base on desired current"
- note added: "3. it is mandatory to add resistor to LDM and VPC when both connected VPACK"
- note added: "BMS BALANCING CIRCUIT"
- note added: "BMS CELL CONNECTOR"
- note added: "BMS CHG & DIS SWITCH"
- note added: "BMS REGULATOR CIRCUIT"
- note added: "BMS Wakeup sequence"
- note added: "Datasheet KA49522A, page 90. Rev 2.08"
- note added: "Ganti aja terminal gapapa"
- note added: "Notes : 1. SRP and SRN Sensing lines have to be drawn side by side on the same PCB layer"
- note added: "Notes : 1. set REGSEL pin=H For REGEXT=3.3V output settings (KA49522A-2101EL-01, page 7,Rev 2.08)"
- note added: "POWER SELECTOR"
- note added: "TMON 1 & 2"
- note added: "TMON internal circuit"
- note added: "insert RVBAT ~ 100ohm for Hotplug protection Insert C (typically about 1uF) for stable voltage"
- note removed: "CELL BALANCING PORT"
- note removed: "CHG & DIS SWITCH"
- note removed: "POWER SELECTOR + LDO"
- note removed: "REGULATOR CIRCUIT"
- company: (none) -> STP OTOMOTIF ITS
- title: (none) -> Nuvoton BMS Board
- moved on the sheet: C10, C11, C12, C23, C36, C37, C38, C39, C40, C41, C42, C43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

Commit message: revision 7 March
Parts:
- removed C11: 100n, Capacitor_SMD:C_0603_1608Metric, symbol Device:C
- removed C37: 1u,0603, Capacitor_SMD:C_0603_1608Metric, symbol Device:C
- removed D24: GREEN_LED, LED_SMD:LED_0603_1608Metric, symbol Device:LED
- removed Q5 (x7), Q6 (x4): NMOS, Package_TO_SOT_SMD:TO-263-2, symbol Simulation_SPICE:NMOS
- removed SW1: SW_SPDT, PROYEK_BMS_NUVOTON:SW_100SP1T1B1M1QEH, symbol Switch:SW_SPDT
- removed SW4: SW_Push, symbol Switch:SW_Push
- removed U6: AP7370-33SA-7, Package_TO_SOT_SMD:SOT-23-3, symbol Regulator_Linear:AP7370-33FDC
- added JP1: Jumper_2_Bridged, Jumper:SolderJumper-2_P1.3mm_Bridged_RoundedPad1.0x1.5mm, symbol Jumper:Jumper_2_Bridged
- added NT1: NetTie_2, NetTie:NetTie-2_SMD_Pad0.5mm, symbol Device:NetTie_2
- added Q6 (x11): NMOS, Package_TO_SOT_SMD:TO-263-2, symbol Device:Q_NMOS_GDS
- added R138, R139, R140, R141, R142, R143, R144, R145, R146, R147, R148: 22, Resistor_SMD:R_0603_1608Metric, symbol Device:R
- added SW1: SW_Push, Button_Switch_SMD:SW_SPST_SKQG_WithStem, symbol Switch:SW_Push
- C23: footprint Capacitor_SMD:C_0805_2012Metric -> Capacitor_SMD:C_0603_1608Metric
- C36: value 1u,0603 -> 100n,0603; JLCPCB Part # C15849 -> C14663
- C49, C50, C51, C52, C53, C54, C55, C56, C57, C58, C59, C60, C61, C62, C63, C64, C65, C66, C67, C68, C69, C70, C71: value 180n -> 1u
- C49: footprint (none) -> Capacitor_SMD:C_0805_2012Metric
- CVBAT1: footprint (none) -> Capacitor_SMD:C_1206_3216Metric
- DVBAT1: value NHP120SFT3G -> US1M; footprint (none) -> Diode_SMD:D_SMA; JLCPCB Part # (none) -> C412437
- J1: footprint (none) -> Connector_PinHeader_2.54mm:PinHeader_1x23_P2.54mm_Vertical
- Q1: symbol Simulation_SPICE:NPN -> Device:Q_NPN_BCE
- Q6: symbol Simulation_SPICE:NMOS -> Device:Q_NMOS_GDS
- R103, R105, R108, R112, R113, R115, R117, R119, R121, R123, R125, R126, R81, R84, R86, R88, R90, R92, R94, R95, R97, R99: value 910 -> 1k
- R132: value 1.2k,0603 -> 22; JLCPCB Part # C22765 -> C23345
- R137: value 75M -> 0
- R2: value 30k -> 0
- R25, R26: footprint Capacitor_SMD:C_0805_2012Metric_Pad1.18x1.45mm_HandSolder -> Capacitor_SMD:C_0603_1608Metric
- RVBAT1, RVBAT2: footprint (none) -> Resistor_SMD:R_1206_3216Metric
- SW3: footprint Button_Switch_THT:SW_CuK_OS102011MA1QN1_SPDT_Angled -> Button_Switch_SMD:SW_SPDT_PCM12
- U1: footprint Package_QFP:HTQFP-64-1EP_10x10mm_P0.5mm_EP5.5x5.5mm_Mask4.4x4.4mm_ThermalVias -> Package_QFP:HTQFP-64-1EP_10x10mm_P0.5mm_EP8x8mm
- Y2: symbol Device:Crystal -> Device:Crystal_GND23
Connections:
- net GNDA is gone; now on net GND: C67.2, CVBAT1.1
- net OSC_0_IN is gone; now on net OSC_IN: C39.2, Y1.2
- net OSC_0_OUT is gone; now on net OSC_OUT: R133.2
- net +3V3: now also C36.1, JP1.2 (B)
- net BMS_3.3V: now also JP1.1 (A)
- net CAN_D+: now also J4.2 (Pin_2); no longer J4.1 (Pin_1)
- net CAN_D-: now also J4.1 (Pin_1); no longer J4.2 (Pin_2)
- net CHG: now also R132.1, R138.1, R139.1, R140.1, R141.1, R142.1; no longer Q6.2 (G)
- net CN4_C22: now also Q6.3 (S), Q6.3 (S), Q6.3 (S), Q6.3 (S), Q6.3 (S); no longer CVBAT1.2, RVBAT2.2, U1.28 (VBAT)
- net DIS: now also R143.1, R144.1, R145.1, R146.1, R147.1, R148.1
- net GND: now also NT1.1; no longer R132.1, R25.2
- net OSC32_IN: now also U4.3 (PC14), Y2.4; no longer Y2.2
- net OSC32_OUT: no longer U4.3 (PC14)
- net REGB: now also Q1.1 (B); no longer Q1.2 (B)
- net REG_SUP: now also Q6.2 (D), Q6.2 (D), Q6.2 (D), Q6.2 (D), Q6.2 (D), Q6.2 (D), Q6.2 (D), Q6.2 (D), Q6.2 (D), Q6.2 (D), Q6.2 (D), Q6.2 (D); no longer Q6.1 (D)
- net USB_5V: now also D25.4 (VCC)
- net VPACK+: now also Q6.3 (S), Q6.3 (S), Q6.3 (S), Q6.3 (S), Q6.3 (S), Q6.3 (S); no longer C2.1, C5.1, R2.1
- net at R132.2: now also Q6.1 (G)
- net at R15.2: now also Q1.2 (C); no longer Q1.1 (C)
- net at R137.1: now also SW1.1
- removed net +5V: C36.1, D25.4 (VCC)
- new net: Q6.1 (G), R145.2
- new net: Q6.1 (G), R147.2
- new net: Q6.1 (G), R138.2
- new net: Q6.1 (G), R139.2
- new net: Q6.1 (G), R148.2
- new net: Q6.1 (G), R144.2
- new net: NT1.2, R25.2
- new net: Q6.1 (G), R143.2
- new net: Q6.1 (G), R146.2
- new net: Q6.1 (G), R140.2
- new net: Q6.1 (G), R142.2
- new net: Q6.1 (G), R141.2
- new net VBAT-P: C2.1, C5.1, CVBAT1.2, R2.1, RVBAT2.2, SW1.2, U1.28 (VBAT)
Other:
- note added: "kept 1uf as spare first"
- note added: "kept 47k as spare first"
- note added: "kept 75M and 30K as spare"
- moved on the sheet: D23, Q6, R75, R76, U2

Commit message: revision 11 march
Parts:
- added C11: 1u, Capacitor_SMD:C_1210_3225Metric, symbol Device:C
- added JP2: SolderJumper_3_Open, symbol Jumper:SolderJumper_3_Open
Connections:
- net BMS_3.3V: now also C11.1
- net GND: now also C11.2
- net VBAT-P: now also JP2.1 (A); no longer C2.1, C5.1, R2.1, SW1.2
- net VPACK+: now also C2.1, C5.1, R2.1, JP2.3 (B)
- new net: JP2.2 (C), SW1.2
